Commit message: Finished Assignment 2

File: body.urdf (robot description, URDF)
Before this commit: robot robot, 2 links, 1 joints
Links:
- removed link Leg
- added link Bleg, mass 1; collision box size=1 1 1; visual box size=1 1 1
- added link Fleg, mass 1; collision box size=1 1 1; visual box size=1 1 1
Joints:
- removed joint Torso_Leg
- added joint Torso_Bleg: type revolute, parent Torso, child Bleg, origin xyz=1 0 1 rpy=0 0 0, axis 0 1 0, limit lower=-3.14159 upper=3.14159 effort=0.0 velocity=0.0
- added joint Torso_Fleg: type revolute, parent Torso, child Fleg, origin xyz=2 0 1 rpy=0 0 0, axis 0 1 0, limit lower=-3.14159 upper=3.14159 effort=0.0 velocity=0.0

Commit message: Step 20 fleg is looking good

File: body.urdf (robot description, URDF)
Before this commit: robot robot, 3 links, 2 joints
Links:
- link Fleg: geometry collision box size=0.2 1 0.2; visual box size=0.2 1 0.2
Joints:
- joint Torso_Fleg: origin xyz=2 0 1 rpy=0 0 0 -> xyz=0 0.5 1 rpy=0 0 0

Commit message: Step 24 bleg is looking good

File: body.urdf (robot description, URDF)
Before this commit: robot robot, 3 links, 2 joints
Links:
- link Bleg: geometry collision box size=0.2 1 0.2; visual box size=0.2 1 0.2
Joints:
- joint Torso_Bleg: origin xyz=1 0 1 rpy=0 0 0 -> xyz=0 -0.5 1 rpy=0 0 0

Commit message: Step 42 Rleg and Lleg both looking good

File: body.urdf (robot description, URDF)
Before this commit: robot robot, 3 links, 2 joints
Links:
- added link Lleg, mass 1; collision box size=1.0 0.2 0.2; visual box size=1.0 0.2 0.2
- added link Rleg, mass 1; collision box size=1.0 0.2 0.2; visual box size=1.0 0.2 0.2
Joints:
- added joint Torso_Lleg: type revolute, parent Torso, child Lleg, origin xyz=-0.5 0 1 rpy=0 0 0, axis 0 1 0, limit lower=-3.14159 upper=3.14159 effort=0.0 velocity=0.0
- added joint Torso_Rleg: type revolute, parent Torso, child Rleg, origin xyz=0.5 0 1 rpy=0 0 0, axis 0 1 0, limit lower=-3.14159 upper=3.14159 effort=0.0 velocity=0.0
- joint Torso_Bleg: axis 0 1 0 -> 1 0 0
- joint Torso_Fleg: axis 0 1 0 -> 1 0 0

Commit message: Step 47 fully formed quadruped

File: body.urdf (robot description, URDF)
Before this commit: robot robot, 5 links, 4 joints
Links:
- added link BackLowerLeg, mass 1; collision box size=0.2 0.2 1; visual box size=0.2 0.2 1
- added link FrontLowerLeg, mass 1; collision box size=0.2 0.2 1; visual box size=0.2 0.2 1
- added link LeftLowerLeg, mass 1; collision box size=0.2 0.2 1; visual box size=0.2 0.2 1
- added link RightLowerLeg, mass 1; collision box size=0.2 0.2 1; visual box size=0.2 0.2 1
Joints:
- added joint Bleg_BackLowerLeg: type revolute, parent Bleg, child BackLowerLeg, origin xyz=0 -1 0 rpy=0 0 0, axis 1 0 0, limit lower=-3.14159 upper=3.14159 effort=0.0 velocity=0.0
- added joint Fleg_FrontLowerLeg: type revolute, parent Fleg, child FrontLowerLeg, origin xyz=0 1 0 rpy=0 0 0, axis 1 0 0, limit lower=-3.14159 upper=3.14159 effort=0.0 velocity=0.0
- added joint Lleg_LeftLowerLeg: type revolute, parent Lleg, child LeftLowerLeg, origin xyz=-1 0 0 rpy=0 0 0, axis 0 1 0, limit lower=-3.14159 upper=3.14159 effort=0.0 velocity=0.0
- added joint Rleg_RightLowerLeg: type revolute, parent Rleg, child RightLowerLeg, origin xyz=1 0 0 rpy=0 0 0, axis 0 1 0, limit lower=-3.14159 upper=3.14159 effort=0.0 velocity=0.0

Commit message: sitting robot

File: body.urdf (robot description, URDF)
Before this commit: robot robot, 9 links, 8 joints
Joints:
- joint Lleg_LeftLowerLeg: axis 0 1 0 -> 0 -1 0
- joint Rleg_RightLowerLeg: axis 0 1 0 -> 0 -1 0
- joint Torso_Lleg: axis 0 1 0 -> 0 -1 0
- joint Torso_Rleg: axis 0 1 0 -> 0 -1 0

Commit message: robot evolves to stay on the platform

File: body.urdf (robot description, URDF)
Before this commit: robot robot, 9 links, 8 joints
Joints:
- joint Torso_Bleg: origin xyz=0 -0.5 1 rpy=0 0 0 -> xyz=0 -0.5 4 rpy=0 0 0
- joint Torso_Fleg: axis 1 0 0 -> -1 0 0; origin xyz=0 0.5 1 rpy=0 0 0 -> xyz=0 0.5 4 rpy=0 0 0
- joint Torso_Lleg: origin xyz=-0.5 0 1 rpy=0 0 0 -> xyz=-0.5 0 4 rpy=0 0 0
- joint Torso_Rleg: axis 0 -1 0 -> 0 1 0; origin xyz=0.5 0 1 rpy=0 0 0 -> xyz=0.5 0 4 rpy=0 0 0

Commit message: initial ab testing commit

File: body.urdf (robot description, URDF)
Before this commit: robot robot, 9 links, 8 joints
Links:
- link BackLowerLeg: geometry collision box size=0.2 0.2 1.5; visual box size=0.2 0.2 1.5
- link FrontLowerLeg: geometry collision box size=0.2 0.2 1.5; visual box size=0.2 0.2 1.5
- link LeftLowerLeg: geometry collision box size=0.2 0.2 1.5; visual box size=0.2 0.2 1.5
- link RightLowerLeg: geometry collision box size=0.2 0.2 1.5; visual box size=0.2 0.2 1.5
Joints:
- joint Torso_Bleg: origin xyz=0 -0.5 4 rpy=0 0 0 -> xyz=0 -0.5 4.5 rpy=0 0 0
- joint Torso_Fleg: origin xyz=0 0.5 4 rpy=0 0 0 -> xyz=0 0.5 4.5 rpy=0 0 0
- joint Torso_Lleg: origin xyz=-0.5 0 4 rpy=0 0 0 -> xyz=-0.5 0 4.5 rpy=0 0 0
- joint Torso_Rleg: origin xyz=0.5 0 4 rpy=0 0 0 -> xyz=0.5 0 4.5 rpy=0 0 0
